File: Type 2280/KiCad/SSD_M2.kicad_pcb (KiCad board)
At the start: 2 copper layers, 22 x 80 mm, 1 part

Commit message: upd
Parts:
- moved JP1 18.6 mm to (1.80, -1.50), turned to 0 degrees
Other:
- outline, holes or cut-outs redrawn
